File: shield.kicad_pcb (KiCad board)
At the start: 2 copper layers, 68.6 x 55.9 mm, 2 parts, among them J1 Conn_01x20, J2 Conn_01x20

Commit message: poop
Parts:
- added J4: 10118193-0001LF, shield_rsrc:FCI_10118193-0001LF, F.Cu at (92.7, 62.4)
- added J5: USB-A-S-X-X-SM2, shield_rsrc:SAMTEC_USB-A-S-X-X-SM2, F.Cu at (73.7, 71.0)
- added R4: 33R, Resistor_SMD:R_0603_1608Metric_Pad0.98x0.95mm_HandSolder, F.Cu at (166.0, 61.5)
- added R5: 33R, Resistor_SMD:R_0603_1608Metric_Pad0.98x0.95mm_HandSolder, F.Cu at (149.8, 76.6)
- added R6: 33R, Resistor_SMD:R_0603_1608Metric_Pad0.98x0.95mm_HandSolder, F.Cu at (149.8, 79.1)
- added R7: 33R, Resistor_SMD:R_0603_1608Metric_Pad0.98x0.95mm_HandSolder, F.Cu at (155.7, 71.0)
- added U1: ATmega328P-A, Package_QFP:TQFP-32_7x7mm_P0.8mm, F.Cu at (147.7, 66.1)
- added U2: MAX4793EUKT, shield_rsrc:SOT95P280X145-5N, F.Cu at (145.0, 74.2)
- added U3: MAX3421EEHJ+T, shield_rsrc:QFP50P700X700X120-32N, F.Cu at (159.1, 65.0)
- added Y1: Crystal, Crystal:Crystal_HC49-U_Vertical, F.Cu at (127.3, 80.4)
- added Y2: CSTNE12M0G550000R0, shield_rsrc:OSC_CSTNE12M0G550000R0, F.Cu at (150.6, 73.6)
Connections:
- J2 pad 19: Net-(J2-Pad19) -> unconnected-(J2-Pad19)

Commit message: pewpewpew
Parts:
- added C1: C, Capacitor_SMD:C_0603_1608Metric_Pad1.08x0.95mm_HandSolder, F.Cu at (87.6, 78.7)
- added C2: C, Capacitor_SMD:C_0603_1608Metric_Pad1.08x0.95mm_HandSolder, F.Cu at (77.5, 78.7)
- added C3: C, Capacitor_SMD:C_0603_1608Metric_Pad1.08x0.95mm_HandSolder, F.Cu at (99.1, 81.3)
- added J3: AVR-ISP-6, Connector_PinHeader_2.54mm:PinHeader_2x03_P2.54mm_Vertical, F.Cu at (78.7, 99.1)
- added R1: R, Resistor_SMD:R_0603_1608Metric_Pad0.98x0.95mm_HandSolder, F.Cu at (72.4, 95.2)
- added R2: R, Resistor_SMD:R_0603_1608Metric_Pad0.98x0.95mm_HandSolder, F.Cu at (97.8, 99.1)
- added R3: R, Resistor_SMD:R_0603_1608Metric_Pad0.98x0.95mm_HandSolder, F.Cu at (99.1, 85.1)
- added SW1: SW_DIP_x01, shield_rsrc:PinHeader_Switch, F.Cu at (91.4, 96.5)
- moved R4 92.7 mm to (74.9, 78.7), turned to 90 degrees
- moved R5 77.5 mm to (72.4, 78.7), turned to 90 degrees
- moved U1 74.7 mm to (76.2, 87.6)
- moved U3 68.7 mm to (92.7, 82.5)
- moved R7 64.3 mm to (91.4, 68.6), turned to 90 degrees
- moved Y1 61.2 mm to (67.3, 92.6), turned to 90 degrees
- moved U2 58.7 mm to (86.4, 74.9), turned to 90 degrees
- moved R6 56.9 mm to (94.0, 68.6), turned to 90 degrees
- moved Y2 52.9 mm to (97.8, 77.5), turned to 135 degrees
Routing:
- net GND: track 0.00 -> 81.5 mm, vias 0 -> 3
- net 5V: track 0.00 -> 51.2 mm, vias 0 -> 1
- net AVR_RESET: track 0.00 -> 46.4 mm, vias 0 -> 1
- net D_PLUS: track 0.00 -> 39.9 mm, vias 0 -> 3
- net H_MOSI: track 0.00 -> 37.4 mm
- net D_MINUS: track 0.00 -> 37.0 mm, vias 0 -> 3
- net H_RESN: track 0.00 -> 31.9 mm, vias 0 -> 2
- net H_MISO: track 0.00 -> 29.0 mm
- net VCC: track 0.00 -> 28.9 mm, vias 0 -> 5
- net H_SCK: track 0.00 -> 26.8 mm, vias 0 -> 1
- net H_SS: track 0.00 -> 23.9 mm, vias 0 -> 2
- net VBUS_COMP: track 0.00 -> 21.8 mm
- net VUSB: track 0.00 -> 12.4 mm
- net VUSB_ON: track 0.00 -> 11.7 mm, vias 0 -> 2
- net FLAG: track 0.00 -> 9.52 mm
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- added copper zone on In2.Cu, net GND
- added copper zone on In1.Cu, net VCC
Other:
- copper layers 2 -> 4

Commit message: save
Parts:
- added J6: Conn_01x04, Connector_PinHeader_2.54mm:PinHeader_1x04_P2.54mm_Vertical, F.Cu at (61.0, 113.0)
- added J7: D7 / TRIG, shield_rsrc:RF2-04A-T-00-50-G, F.Cu at (78.7, 111.8)
- moved Y1 2.54 mm to (64.8, 92.6)
- moved C1 1.27 mm to (86.4, 78.7)
Connections:
- U1 pad 11: unconnected-(U1-Pad11) -> PIN_TRIG
- U1 pad 30: unconnected-(U1-Pad30) -> RXD
- U1 pad 31: unconnected-(U1-Pad31) -> TXD
Routing:
- net RXD: track 0.00 -> 34.6 mm, vias 0 -> 1
- net TXD: track 0.00 -> 34.1 mm, vias 0 -> 1
- net PIN_TRIG: track 0.00 -> 24.9 mm, vias 0 -> 1
- net Net-(J5-PadS1): track 0.00 -> 14.5 mm
- net VCC: track 28.9 -> 41.9 mm
- net Net-(J4-PadS1): track 0.00 -> 8.96 mm
- net Net-(U1-Pad7): track 5.42 -> 7.96 mm
- net Net-(U1-Pad8): track 5.55 -> 8.09 mm
- net GND: track 81.5 -> 82.4 mm
Other:
- board text added: "RXD"
- board text added: "TXD"
- board text added: "VCC"

Commit message: decoupling
Parts:
- added C4: C, Capacitor_SMD:C_0603_1608Metric_Pad1.08x0.95mm_HandSolder, F.Cu at (67.7, 80.0)
- added C5: C, Capacitor_SMD:C_0603_1608Metric_Pad1.08x0.95mm_HandSolder, F.Cu at (67.7, 82.5)
- J7: value D7 / TRIG -> Conn_Coaxial
Connections:
- J7 pad 3: GND -> (no net)
- J7 pad 4: GND -> (no net)
- J7 pad 5: GND -> (no net)
Routing:
- net GND: track 82.4 -> 89.5 mm
- net VCC: track 41.9 -> 47.0 mm, vias 5 -> 6

Commit message: dont let your dreams be memes
Parts:
- added C6: C, Capacitor_SMD:C_0603_1608Metric_Pad1.08x0.95mm_HandSolder, F.Cu at (85.1, 82.5)
- added C7: C, Capacitor_SMD:C_0603_1608Metric_Pad1.08x0.95mm_HandSolder, F.Cu at (85.1, 85.1)
Routing:
- net GND: track 89.5 -> 96.3 mm
- net VCC: track 47.0 -> 51.7 mm, vias 6 -> 7
Changed lines of the file:
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@@
+    )
+  )
+  (footprint "Capacitor_SMD:C_0603_1608Metric_Pad1.08x0.95mm_HandSolder" (layer "F.Cu")
+    (at 85.09 82.55 180)
+    (descr "Capacitor SMD 0603 (1608 Metric), square (rectangular) end terminal, IPC_7351 nominal with elongated pad for handsoldering. (Body size source: IPC-SM-782 page 76, https://www.pcb-3d.com/wordpress/wp-content/uploads/ipc-sm-782a_amendment_1_and_2.pdf), generated with kicad-footprint-generator")
+    (tags "capacitor handsolder")
+    (property "Sheetfile" "shield.kicad_sch")
+    (property "Sheetname" "")
+    (attr smd)
+    (fp_text reference "C6" (at 0 -3.81) (layer "F.SilkS")
+      (effects (font (size 1 1) (thickness 0.15)))
+    )
+    (fp_text value "C" (at 0 1.43) (layer "F.Fab")
+      (effects (font (size 1 1) (thickness 0.15)))
+    )
+    (fp_text user "${REFERENCE}" (at 0 0) (layer "F.Fab")
+      (effects (font (size 0.4 0.4) (thickness 0.06)))
+    )
+    (fp_line (start -0.146267 0.51) (end 0.146267 0.51) (layer "F.SilkS") (width 0.12))
+    (fp_line (start -0.146267 -0.51) (end 0.146267 -0.51) (layer "F.SilkS") (width 0.12))
+    (fp_line (start -1.65 -0.73) (end 1.65 -0.73) (layer "F.CrtYd") (width 0.05))
+    (fp_line (start -1.65 0.73) (end -1.65 -0.73) (layer "F.CrtYd") (width 0.05))
+    (fp_line (start 1.65 -0.73) (end 1.65 0.73) (layer "F.CrtYd") (width 0.05))
+    (fp_line (start 1.65 0.73) (end -1.65 0.73) (layer "F.CrtYd") (width 0.05))
+    (fp_line (start -0.8 -0.4) (end 0.8 -0.4) (layer "F.Fab") (width 0.1))
+    (fp_line (start -0.8 0.4) (end -0.8 -0.4) (layer "F.Fab") (width 0.1))
+    (fp_line (start 0.8 0.4) (end -0.8 0.4) (layer "F.Fab") (width 0.1))
+    (fp_line (start 0.8 -0.4) (end 0.8 0.4) (layer "F.Fab") (width 0.1))
+    (pad "1" smd roundrect (at -0.8625 0 180) (size 1.075 0.95) (layers "F.Cu" "F.Paste" "F.Mask") (roundrect_rratio 0.25)
+      (net 53 "VCC") (pintype "passive"))
+    (pad "2" smd roundrect (at 0.8625 0 180) (size 1.075 0.95) (layers "F.Cu" "F.Paste" "F.Mask") (roundrect_rratio 0.25)
+      (net 1 "GND") (pintype "passive"))
+    (model "${KICAD6_3DMODEL_DIR}/Capacitor_SMD.3dshapes/C_0603_1608Metric.wrl"
+      (offset (xyz 0 0 0))
+      (scale (xyz 1 1 1))
+      (rotate (xyz 0 0 0))
     )
   )
@@
   )
   (footprint "Capacitor_SMD:C_0603_1608Metric_Pad1.08x0.95mm_HandSolder" (layer "F.Cu")
+    (at 85.09 85.06 180)
+    (descr "Capacitor SMD 0603 (1608 Metric), square (rectangular) end terminal, IPC_7351 nominal with elongated pad for handsoldering. (Body size source: IPC-SM-782 page 76, https://www.pcb-3d.com/wordpress/wp-content/uploads/ipc-sm-782a_amendment_1_and_2.pdf), generated with kicad-footprint-generator")
+    (tags "capacitor handsolder")
+    (property "Sheetfile" "shield.kicad_sch")
+    (property "Sheetname" "")
+    (attr smd)
+    (fp_text reference "C7" (at 0 -2.57) (layer "F.SilkS")
+      (effects (font (size 1 1) (thickness 0.15)))
+    )
+    (fp_text value "C" (at 0 1.43) (layer "F.Fab")
+      (effects (font (size 1 1) (thickness 0.15)))
+    )
+    (fp_text user "${REFERENCE}" (at 0 0) (layer "F.Fab")
+      (effects (font (size 0.4 0.4) (thickness 0.06)))
+    )
+    (fp_line (start -0.146267 -0.51) (end 0.146267 -0.51) (layer "F.SilkS") (width 0.12))
+    (fp_line (start -0.146267 0.51) (end 0.146267 0.51) (layer "F.SilkS") (width 0.12))
+    (fp_line (start -1.65 0.73) (end -1.65 -0.73) (layer "F.CrtYd") (width 0.05))
+    (fp_line (start -1.65 -0.73) (end 1.65 -0.73) (layer "F.CrtYd") (width 0.05))
+    (fp_line (start 1.65 -0.73) (end 1.65 0.73) (layer "F.CrtYd") (width 0.05))
+    (fp_line (start 1.65 0.73) (end -1.65 0.73) (layer "F.CrtYd") (width 0.05))
+    (fp_line (start -0.8 -0.4) (end 0.8 -0.4) (layer "F.Fab") (width 0.1))
+    (fp_line (start 0.8 0.4) (end -0.8 0.4) (layer "F.Fab") (width 0.1))
+    (fp_line (start -0.8 0.4) (end -0.8 -0.4) (layer "F.Fab") (width 0.1))
+    (fp_line (start 0.8 -0.4) (end 0.8 0.4) (layer "F.Fab") (width 0.1))
+    (pad "1" smd roundrect (at -0.8625 0 180) (size 1.075 0.95) (layers "F.Cu" "F.Paste" "F.Mask") (roundrect_rratio 0.25)
+      (net 53 "VCC") (pintype "passive"))
+    (pad "2" smd roundrect (at 0.8625 0 180) (size 1.075 0.95) (layers "F.Cu" "F.Paste" "F.Mask") (roundrect_rratio 0.25)
+      (net 1 "GND") (pintype "passive"))
+    (model "${KICAD6_3DMODEL_DIR}/Capacitor_SMD.3dshapes/C_0603_1608Metric.wrl"
+      (offset (xyz 0 0 0))
+      (scale (xyz 1 1 1))
+      (rotate (xyz 0 0 0))
+    )
+  )
+  (footprint "Capacitor_SMD:C_0603_1608Metric_Pad1.08x0.95mm_HandSolder" (layer "F.Cu")
     (at 67.7175 80.04 180)
     (descr "Capacitor SMD 0603 (1608 Metric), square (rectangular) end terminal, IPC_7351 nominal with elongated pad for handsoldering. (Body size source: IPC-SM-782 page 76, https://www.pcb-3d.com/wordpress/wp-content/uploads/ipc-sm-782a_amendment_1_and_2.pdf), generated with kicad-footprint-generator")
@@
     (fp_circle (center -2.22 0) (end -2.12 0) (layer "F.SilkS") (width 0.2) (fill none))
     (fp_line (start -1.85 -1.2) (end 1.85 -1.2) (layer "F.CrtYd") (width 0.05))
+    (fp_line (start -1.85 1.2) (end -1.85 -1.2) (layer "F.CrtYd") (width 0.05))
+    (fp_line (start 1.85 -1.2) (end 1.85 1.2) (layer "F.CrtYd") (width 0.05))
     (fp_line (start 1.85 1.2) (end -1.85 1.2) (layer "F.CrtYd") (width 0.05))
-    (fp_line (start 1.85 -1.2) (end 1.85 1.2) (layer "F.CrtYd") (width 0.05))
-    (fp_line (start -1.85 1.2) (end -1.85 -1.2) (layer "F.CrtYd") (width 0.05))
+    (fp_line (start 1.6 -0.65) (end 1.6 0.65) (layer "F.Fab") (width 0.127))
     (fp_line (start 1.6 0.65) (end -1.6 0.65) (layer "F.Fab") (width 0.127))
-    (fp_line (start 1.6 -0.65) (end 1.6 0.65) (layer "F.Fab") (width 0.127))
     (fp_line (start -1.6 -0.65) (end -1.6 0.65) (layer "F.Fab") (width 0.127))
     (fp_line (start -1.6 -0.65) (end 1.6 -0.65) (layer "F.Fab") (width 0.127))
@@
   (segment (start 85.4975 78.74) (end 86.36 77.8775) (width 0.25) (layer "F.Cu") (net 1))
   (segment (start 66.855 80.04) (end 66.855 82.55) (width 0.25) (layer "F.Cu") (net 1))
+  (segment (start 85.4975 81.28) (end 84.2275 82.55) (width 0.25) (layer "F.Cu") (net 1))
   (segment (start 85.09 78.74) (end 81.28 78.74) (width 0.25) (layer "F.Cu") (net 1))
   (segment (start 93.966955 71.844511) (end 88.354511 71.844511) (width 0.25) (layer "F.Cu") (net 1))
@@
   (segment (start 78.81 86.43) (end 79.61 87.23) (width 0.25) (layer "F.Cu") (net 1))
   (segment (start 95.89 83.3) (end 97.9025 83.3) (width 0.25) (layer "F.Cu") (net 1))
+  (segment (start 85.4975 78.74) (end 85.4975 81.28) (width 0.25) (layer "F.Cu") (net 1))
   (segment (start 86.36 77.8775) (end 86.36 76.175) (width 0.25) (layer "F.Cu") (net 1))
   (segment (start 99.9225 81.28) (end 101.6 81.28) (width 0.25) (layer "F.Cu") (net 1))
@@
   (segment (start 88.354511 71.844511) (end 87.63 71.12) (width 0.25) (layer "F.Cu") (net 1))
   (segment (start 70.825489 86.630489) (end 71.025978 86.43) (width 0.25) (layer "F.Cu") (net 1))
+  (segment (start 84.2275 85.06) (end 84.2275 82.55) (width 0.25) (layer "F.Cu") (net 1))
   (segment (start 70.9 86.43) (end 70.16 85.69) (width 0.25) (layer "F.Cu") (net 1))
   (via (at 87.63 71.12) (size 0.8) (drill 0.4) (layers "F.Cu" "B.Cu") (net 1))
@@
   (segment (start 91.44 80.01) (end 91.44 71.12) (width 0.25) (layer "In2.Cu") (net 50))
   (segment (start 97.79 98.1475) (end 97.79 96.52) (width 0.25) (layer "F.Cu") (net 53))
+  (segment (start 85.9525 85.06) (end 85.9525 82.55) (width 0.25) (layer "F.Cu") (net 53))
   (segment (start 73.73 88.83) (end 74.102011 88.457989) (width 0.25) (layer "F.Cu") (net 53))
   (segment (start 74.337011 87.23) (end 71.95 87.23) (width 0.25) (layer "F.Cu") (net 53))
@@
   (segment (start 74.737011 87.63) (end 74.737011 87.822989) (width 0.25) (layer "F.Cu") (net 53))
   (segment (start 88.657621 81.3) (end 87.63 80.272379) (width 0.25) (layer "F.Cu") (net 53))
+  (segment (start 85.9525 82.55) (end 86.36 82.55) (width 0.25) (layer "F.Cu") (net 53))
   (segment (start 89.53 81.3) (end 88.657621 81.3) (width 0.25) (layer "F.Cu") (net 53))
   (segment (start 74.737011 87.63) (end 76.737011 89.63) (width 0.25) (layer "F.Cu") (net 53))
+  (segment (start 86.36 82.55) (end 87.63 83.82) (width 0.25) (layer "F.Cu") (net 53))
   (segment (start 87.63 79.1475) (end 87.2225 78.74) (width 0.25) (layer "F.Cu") (net 53))
   (segment (start 74.737011 87.63) (end 74.337011 87.23) (width 0.25) (layer "F.Cu") (net 53))
@@
   (via (at 87.63 80.01) (size 0.8) (drill 0.4) (layers "F.Cu" "B.Cu") (net 53))
   (via (at 68.58 85.09) (size 0.8) (drill 0.4) (layers "F.Cu" "B.Cu") (free) (net 53))
+  (via (at 87.63 83.82) (size 0.8) (drill 0.4) (layers "F.Cu" "B.Cu") (free) (net 53))
   (via (at 69.85 97.79) (size 0.8) (drill 0.4) (layers "F.Cu" "B.Cu") (free) (net 53))
   (via (at 97.79 96.52) (size 0.8) (drill 0.4) (layers "F.Cu" "B.Cu") (free) (net 53))
